Commit message: updates for jazzy to make it work in the simulation

File: robotiq_description/urdf/robotiq_2f_140.xacro (robot description, xacro)
@@ -154,6 +154,8 @@
     <xacro:finger_joints prefix="${prefix}" fingerprefix="left" reflect="1.0"/>
   </xacro:macro>
-  <xacro:macro name="right_outer_knuckle_joint" params="prefix">
-    <joint name="${prefix}right_outer_knuckle_joint" type="revolute">
+  <xacro:macro name="right_outer_knuckle_joint" params="prefix sim_gazebo:=false">
+    <!-- Gazebo velocity-driven mimics can stick at a redundant joint stop.
+         In simulation, the bounded master joint supplies the motion limits. -->
+    <joint name="${prefix}right_outer_knuckle_joint" type="${'continuous' if sim_gazebo else 'revolute'}">
       <origin xyz="0 0.030601 0.054905" rpy="${pi / 2 + .725} 0 ${pi}" />
       <parent link="${prefix}robotiq_140_base_link" />

File: robotiq_description/urdf/robotiq_2f_140_macro.urdf.xacro (robot description, xacro)
@@ -77,5 +77,5 @@
       <xacro:finger_links prefix="${prefix}" fingerprefix="right" stroke="140"/>
       <xacro:finger_joint prefix="${prefix}"/>
-      <xacro:right_outer_knuckle_joint prefix="${prefix}"/>
+      <xacro:right_outer_knuckle_joint prefix="${prefix}" sim_gazebo="${sim_gazebo}"/>
     </xacro:macro>
 </robot>

File: robotiq_description/urdf/robotiq_2f_85_macro.urdf.xacro (robot description, xacro)
@@ -232,4 +232,8 @@
             <xacro:insert_block name="origin" />
         </joint>
+        <!-- Gazebo's position/mimic velocity motors need headroom for tracking
+             corrections. The 0.5 rad/s hardware limit causes follower divergence
+             even for a 0.1 rad goal. Keep all physical position stops and use the
+             original velocity limit outside Gazebo. -->
         <joint name="${prefix}robotiq_85_left_knuckle_joint" type="revolute">
             <parent link="${prefix}robotiq_85_base_link" />
@@ -237,5 +241,5 @@
             <axis xyz="0 -1 0" />
             <origin xyz="0.03060114 0.0 0.05490452" rpy="0 0 0" />
-            <limit lower="0.0" upper="0.8" velocity="0.5" effort="50" />
+            <limit lower="0.0" upper="0.8" velocity="${10.0 if sim_gazebo else 0.5}" effort="50" />
         </joint>
         <joint name="${prefix}robotiq_85_right_knuckle_joint" type="revolute">
@@ -244,5 +248,5 @@
             <axis xyz="0 -1 0" />
             <origin xyz="-0.03060114 0.0 0.05490452" rpy="0 0 0" />
-            <limit lower="-0.8" upper="0.0" velocity="0.5" effort="50" />
+            <limit lower="-0.8" upper="0.0" velocity="${10.0 if sim_gazebo else 0.5}" effort="50" />
             <mimic joint="${prefix}robotiq_85_left_knuckle_joint" multiplier="-1" />
         </joint>
@@ -263,5 +267,5 @@
             <origin xyz="0.0127 0.0 0.06142" rpy="0 0 0" />
             <mimic joint="${prefix}robotiq_85_left_knuckle_joint" />
-            <limit lower="0.0" upper="0.8" velocity="0.5" effort="50" />
+            <limit lower="0.0" upper="0.8" velocity="${10.0 if sim_gazebo else 0.5}" effort="50" />
         </joint>
         <joint name="${prefix}robotiq_85_right_inner_knuckle_joint" type="revolute">
@@ -271,5 +275,5 @@
             <origin xyz="-0.0127 0.0 0.06142" rpy="0 0 0" />
             <mimic joint="${prefix}robotiq_85_left_knuckle_joint" multiplier="-1" />
-            <limit lower="-0.8" upper="0.0" velocity="0.5" effort="50" />
+            <limit lower="-0.8" upper="0.0" velocity="${10.0 if sim_gazebo else 0.5}" effort="50" />
         </joint>
         <joint name="${prefix}robotiq_85_left_finger_tip_joint" type="revolute">
@@ -279,5 +283,5 @@
             <origin xyz="0.00563134 0.0 0.04718515" rpy="0 0 0" />
             <mimic joint="${prefix}robotiq_85_left_knuckle_joint" multiplier="-1" />
-            <limit lower="-0.8" upper="0.0" velocity="0.5" effort="50" />
+            <limit lower="-0.8" upper="0.0" velocity="${10.0 if sim_gazebo else 0.5}" effort="50" />
         </joint>
         <joint name="${prefix}robotiq_85_right_finger_tip_joint" type="revolute">
@@ -287,5 +291,5 @@
             <origin xyz="-0.00563134 0.0 0.04718515" rpy="0 0 0" />
             <mimic joint="${prefix}robotiq_85_left_knuckle_joint" />
-            <limit lower="0.0" upper="0.8" velocity="0.5" effort="50" />
+            <limit lower="0.0" upper="0.8" velocity="${10.0 if sim_gazebo else 0.5}" effort="50" />
         </joint>
     </xacro:macro>
